File: watering-system.kicad_pcb (KiCad board)
At the start: 2 copper layers, 1 part, among them U1 NodeMCU_1.0_(ESP-12E)

Commit message: feat: add finished complete DRC approved schematic
Parts:
- added D1: 1N4007, Diode_THT:D_DO-41_SOD81_P10.16mm_Horizontal, F.Cu at (175.8, 101.6)
- added D2: LD271, LED_THT:LED_D5.0mm_IRGrey, F.Cu at (168.9, 103.2)
- added D3: LD271, LED_THT:LED_D5.0mm_IRGrey, F.Cu at (168.9, 110.7)
- added D4: 1N4007, Diode_THT:D_DO-41_SOD81_P10.16mm_Horizontal, F.Cu at (175.8, 105.8)
- added K2: DIPxx-1Cxx-51x, Relay_THT:Relay_StandexMeder_DIP_LowProfile, F.Cu at (168.1, 81.1)
- added K3: DIPxx-1Cxx-51x, Relay_THT:Relay_StandexMeder_DIP_LowProfile, F.Cu at (178.9, 81.1)
- added Q1: 2N2219, Package_TO_SOT_THT:TO-39-3, F.Cu at (158.4, 83.5)
- added Q2: 2N2219, Package_TO_SOT_THT:TO-39-3, F.Cu at (158.4, 94.4)
Connections:
- U1 pad 1: unconnected-(U1-A0(ADC0)-Pad1) -> /ANALOGUE_IN
- U1 pad 10: unconnected-(U1-GND-Pad10) -> GND
- U1 pad 11: unconnected-(U1-3.3V-Pad11) -> +3V3
- U1 pad 14: unconnected-(U1-GND-Pad14) -> GND
- U1 pad 15: unconnected-(U1-VIN-Pad15) -> +5V
- U1 pad 16: unconnected-(U1-3.3V-Pad16) -> +3V3
- U1 pad 17: unconnected-(U1-GND-Pad17) -> GND
- U1 pad 20: unconnected-(U1-D8(GPIO15)-Pad20) -> /ADC_S2
- U1 pad 21: unconnected-(U1-D7(GPIO13)-Pad21) -> /ADC_S1
- U1 pad 22: unconnected-(U1-D6(GPIO12)-Pad22) -> /ADC_S0
- U1 pad 23: unconnected-(U1-D5(GPIO14)-Pad23) -> /TEMP_ONE_WIRE
- U1 pad 24: unconnected-(U1-GND-Pad24) -> GND
- U1 pad 25: unconnected-(U1-3.3V-Pad25) -> +3V3
- U1 pad 26: unconnected-(U1-D4(GPIO2)-Pad26) -> /ULTRASONIC_ECHO
- U1 pad 27: unconnected-(U1-D3(GPIO0)-Pad27) -> /ULTRASONIC_TRIG
- U1 pad 28: unconnected-(U1-D2(GPIO4)-Pad28) -> /PIR
- U1 pad 29: unconnected-(U1-D1(GPIO5)-Pad29) -> /PUMP_1
- U1 pad 30: unconnected-(U1-D0(GPIO16)-Pad30) -> /PUMP_0
