File: watering-system.kicad_sch (KiCad schematic)
At the start: 0 parts

Commit message: feat: Add final pinout of ESP8266 Breakout Board
Confirmed working with Home-Lab-Containers repo and Home Assistant
Parts:
- added C1: 100nF, symbol Device:C
- added C2: 100uF, symbol Device:C_Polarized
- added J1: Conn_01x04_Socket, symbol Connector:Conn_01x04_Socket
- added J2, J3: Conn_01x03_Socket, symbol Connector:Conn_01x03_Socket
- added U1: NodeMCU_1.0_(ESP-12E), ESP8266:NodeMCU-LoLinV3, symbol ESP8266:NodeMCU_1.0_(ESP-12E)
Connections:
- new net +3V3: J1.1 (Pin_1), J2.1 (Pin_1), J3.1 (Pin_1), U1.11 (3.3V), U1.16 (3.3V), U1.25 (3.3V)
- new net +5V: C1.1, C2.1, U1.15 (VIN)
- new net ADC_S0: U1.22 (D6(GPIO12))
- new net ADC_S1: U1.21 (D7(GPIO13))
- new net ADC_S2: U1.20 (D8(GPIO15))
- new net ANALOGUE_IN: U1.1 (A0(ADC0))
- new net ECHO: U1.26 (D4(GPIO2))
- new net GND: C1.2, C2.2, J1.4 (Pin_4), J2.3 (Pin_3), J3.3 (Pin_3), U1.10 (GND), U1.14 (GND), U1.17 (GND), U1.24 (GND)
- new net PIR: U1.28 (D2(GPIO4))
- new net PIR_0: J2.2 (Pin_2)
- new net PIR_1: J3.2 (Pin_2)
- new net PUMP_0: U1.30 (D0(GPIO16))
- new net PUMP_1: U1.29 (D1(GPIO5))
- new net RX: J1.3 (Pin_3)
- new net TEMP: U1.23 (D5(GPIO14))
- new net TRIG: U1.27 (D3(GPIO0))
- new net TX: J1.2 (Pin_2)

Commit message: feat: add finished complete DRC approved schematic
Parts:
- removed J1: Conn_01x04_Socket, symbol Connector:Conn_01x04_Socket
- removed J2, J3: Conn_01x03_Socket, symbol Connector:Conn_01x03_Socket
- added D1, D4: 1N4148, Diode_THT:D_DO-41_SOD81_P10.16mm_Horizontal, symbol Diode:1N4007
- added D2, D3: LD271, LED_THT:LED_D5.0mm_IRGrey, symbol LED:LD271
- added J1: Barrel_Jack, symbol Connector:Barrel_Jack
- added J2: Conn_01x05_Socket, symbol Connector:Conn_01x05_Socket
- added J3: Conn_01x15_Socket, symbol Connector:Conn_01x15_Socket
- added J4: Conn_01x04_Socket, symbol Connector:Conn_01x04_Socket
- added K2, K3: DIPxx-1Cxx-51x, Relay_THT:Relay_StandexMeder_DIP_LowProfile, symbol Relay:DIPxx-1Cxx-51x
- added Q1, Q2: 2N2219, Package_TO_SOT_THT:TO-39-3, symbol Transistor_BJT:2N2219
- added R1: R, symbol Device:R
- added R2, R5: 330, symbol Device:R
- added R3, R4: 1K, symbol Device:R
- added R6, R7: 100, symbol Device:R
- added R8: 4.7K, symbol Device:R
- added U2: 74HC4051, symbol 74xx:74HC4051
- added U3: YAAJ_DCDC_StepDown_LM2596, symbol yaaj_dcdc_stepdown_lm2596:YAAJ_DCDC_StepDown_LM2596
Connections:
- net +3V3: now also J2.1 (Pin_1), J3.1 (Pin_1), J4.1 (Pin_1), R8.1
- net +5V: now also D1.1 (K), D4.1 (K), K2.6, K3.6, R3.2, R4.2, U2.16 (VCC), U3.4 (Vout)
- net ADC_S0: now also U2.11 (S0)
- net ADC_S1: now also U2.10 (S1)
- net ADC_S2: now also U2.9 (S2)
- net ANALOGUE_IN: now also U2.3 (A)
- net GND: now also J1.2, J2.5 (Pin_5), J3.2 (Pin_2), J3.4 (Pin_4), J3.6 (Pin_6), J4.4 (Pin_4), Q1.1 (E), Q2.1 (E), R1.2, R6.1, R7.1, U2.6 (~{E}), U2.7 (VEE), U2.8 (GND), U3.2 (GND), U3.3 (GND)
- net PIR: now also J2.3 (Pin_3)
- net PUMP_0: now also R2.1
- net PUMP_1: now also R5.1
- net RX: now also U1.19 (RX(DPIO3)), J4.3 (Pin_3)
- net TX: now also U1.18 (TX(GPIO1)), J4.2 (Pin_2)
- net ECHO renamed ULTRASONIC_ECHO
- net ULTRASONIC_ECHO: now also J3.8 (Pin_8)
- net TEMP renamed TEMP_ONE_WIRE
- net TEMP_ONE_WIRE: now also J3.10 (Pin_10), R8.2
- net TRIG renamed ULTRASONIC_TRIG
- net ULTRASONIC_TRIG: now also J3.7 (Pin_7)
- new net: Q1.2 (B), R2.2, R7.2
- new net: D1.2 (A), D2.1 (K), K2.2, Q1.3 (C)
- new net: D3.1 (K), D4.2 (A), K3.2, Q2.3 (C)
- new net: D3.2 (A), R4.1
- new net: Q2.2 (B), R5.2, R6.2
- new net: D2.2 (A), R3.1
- new net MUX_A7_IN: J3.15 (Pin_15), U2.4 (A7)
- new net PUMP_PWR_0: J3.3 (Pin_3), K2.14
- new net PUMP_PWR_1: J3.5 (Pin_5), K3.14
- new net RESISTIVE_MOISTURE: J2.4 (Pin_4), U2.15 (A2)
- new net VCC: J1.1, K2.7, K2.8, K3.7, K3.8, U3.1 (Vin)
- new net capacitive_moisture_0: J3.11 (Pin_11), U2.12 (A3)
- new net capacitive_moisture_1: J3.12 (Pin_12), U2.1 (A4)
- new net capacitive_moisture_2: J3.13 (Pin_13), U2.5 (A5)
- new net capacitive_moisture_3: J3.14 (Pin_14), U2.2 (A6)
- new net light_sensor_0: J2.2 (Pin_2), R1.1, U2.13 (A0)
- new net light_sensor_1: J3.9 (Pin_9), U2.14 (A1)
- no-connect marks 0 -> 12
Other:
- title: (none) -> Outdoor Watering System Main Board
- moved on the sheet: C1, C2
