File: main-board/main-board.kicad_sch (KiCad schematic)
At the start: 25 parts, among them J1 Barrel_Jack, J2 Conn_01x05_Socket, J3 Conn_01x15_Socket, J4 Conn_01x04_Socket, K2 DIPxx-1Cxx-51x, K3 DIPxx-1Cxx-51x, Q1 2N2219, Q2 2N2219, U1 NodeMCU_1.0_(ESP-12E), U2 74HC4051, U3 YAAJ_DCDC_StepDown_LM2596

Commit message: feat: split hardware into Main Board and Connector Board projects
Other:
- title: Outdoor Watering System Main Board -> Main Board
Changed lines of the file:
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@@
 	(paper "A4")
 	(title_block
-		(title "Outdoor Watering System Main Board")
+		(title "Main Board")
 		(date "2026-09-18")
 		(rev "See GitHub")
@@
 		)
 		(instances
-			(project "watering-system"
+			(project "main-board"
 				(path "/37f9ca20-4a6d-426d-a8d5-c655e0adba86"
 					(reference "#PWR04")
@@
 		)
 		(instances
-			(project "watering-system"
+			(project "main-board"
 				(path "/37f9ca20-4a6d-426d-a8d5-c655e0adba86"
 					(reference "R2")
@@
 		)
 		(instances
-			(project "watering-system"
+			(project "main-board"
 				(path "/37f9ca20-4a6d-426d-a8d5-c655e0adba86"
 					(reference "K2")
@@
 		)
 		(instances
-			(project "watering-system"
+			(project "main-board"
 				(path "/37f9ca20-4a6d-426d-a8d5-c655e0adba86"
 					(reference "#PWR05")
@@
 		)
 		(instances
-			(project "watering-system"
+			(project "main-board"
 				(path "/37f9ca20-4a6d-426d-a8d5-c655e0adba86"
 					(reference "#PWR022")
@@
 		)
 		(instances
-			(project "watering-system"
+			(project "main-board"
 				(path "/37f9ca20-4a6d-426d-a8d5-c655e0adba86"
 					(reference "C2")
@@
 		)
 		(instances
-			(project "watering-system"
+			(project "main-board"
 				(path "/37f9ca20-4a6d-426d-a8d5-c655e0adba86"
 					(reference "#PWR011")
@@
 		)
 		(instances
-			(project "watering-system"
+			(project "main-board"
 				(path "/37f9ca20-4a6d-426d-a8d5-c655e0adba86"
 					(reference "U3")
@@
 		)
 		(instances
-			(project "watering-system"
+			(project "main-board"
 				(path "/37f9ca20-4a6d-426d-a8d5-c655e0adba86"
 					(reference "#PWR016")
@@
 		)
 		(instances
-			(project "watering-system"
+			(project "main-board"
 				(path "/37f9ca20-4a6d-426d-a8d5-c655e0adba86"
 					(reference "D3")
@@
 		)
 		(instances
-			(project "watering-system"
+			(project "main-board"
 				(path "/37f9ca20-4a6d-426d-a8d5-c655e0adba86"
 					(reference "#PWR010")
@@
 		)
 		(instances
-			(project "watering-system"
+			(project "main-board"
 				(path "/37f9ca20-4a6d-426d-a8d5-c655e0adba86"
 					(reference "#PWR09")
@@
 		)
 		(instances
-			(project "watering-system"
+			(project "main-board"
 				(path "/37f9ca20-4a6d-426d-a8d5-c655e0adba86"
 					(reference "R1")
@@
 		)
 		(instances
-			(project "watering-system"
+			(project "main-board"
 				(path "/37f9ca20-4a6d-426d-a8d5-c655e0adba86"
 					(reference "U1")
@@
 		)
 		(instances
-			(project "watering-system"
+			(project "main-board"
 				(path "/37f9ca20-4a6d-426d-a8d5-c655e0adba86"
 					(reference "#PWR029")
@@
 		)
 		(instances
-			(project "watering-system"
+			(project "main-board"
 				(path "/37f9ca20-4a6d-426d-a8d5-c655e0adba86"
 					(reference "#PWR014")
@@
 		)
 		(instances
-			(project "watering-system"
+			(project "main-board"
 				(path "/37f9ca20-4a6d-426d-a8d5-c655e0adba86"
 					(reference "#PWR030")
@@
 		)
 		(instances
-			(project "watering-system"
+			(project "main-board"
 				(path "/37f9ca20-4a6d-426d-a8d5-c655e0adba86"
 					(reference "#PWR019")
@@
 		)
 		(instances
-			(project "watering-system"
+			(project "main-board"
 				(path "/37f9ca20-4a6d-426d-a8d5-c655e0adba86"
 					(reference "J1")
@@
 		)
 		(instances
-			(project "watering-system"
+			(project "main-board"
 				(path "/37f9ca20-4a6d-426d-a8d5-c655e0adba86"
 					(reference "J2")
@@
 		)
 		(instances
-			(project "watering-system"
+			(project "main-board"
 				(path "/37f9ca20-4a6d-426d-a8d5-c655e0adba86"
 					(reference "Q1")
@@
 		)
 		(instances
-			(project "watering-system"
+			(project "main-board"
 				(path "/37f9ca20-4a6d-426d-a8d5-c655e0adba86"
 					(reference "#PWR032")
@@
 		)
 		(instances
-			(project "watering-system"
+			(project "main-board"
 				(path "/37f9ca20-4a6d-426d-a8d5-c655e0adba86"
 					(reference "#PWR06")
@@
 		)
 		(instances
-			(project "watering-system"
+			(project "main-board"
 				(path "/37f9ca20-4a6d-426d-a8d5-c655e0adba86"
 					(reference "C1")
@@
 		)
 		(instances
-			(project "watering-system"
+			(project "main-board"
 				(path "/37f9ca20-4a6d-426d-a8d5-c655e0adba86"
 					(reference "Q2")
@@
 		)
 		(instances
-			(project "watering-system"
+			(project "main-board"
 				(path "/37f9ca20-4a6d-426d-a8d5-c655e0adba86"
 					(reference "R4")
@@
 		)
 		(instances
-			(project "watering-system"
+			(project "main-board"
 				(path "/37f9ca20-4a6d-426d-a8d5-c655e0adba86"
 					(reference "#PWR02")
@@
 		)
 		(instances
-			(project "watering-system"
+			(project "main-board"
 				(path "/37f9ca20-4a6d-426d-a8d5-c655e0adba86"
 					(reference "R3")
@@
 		)
 		(instances
-			(project "watering-system"
+			(project "main-board"
 				(path "/37f9ca20-4a6d-426d-a8d5-c655e0adba86"
 					(reference "#PWR013")
@@
 		)
 		(instances
-			(project "watering-system"
+			(project "main-board"
 				(path "/37f9ca20-4a6d-426d-a8d5-c655e0adba86"
 					(reference "#PWR017")
@@
 		)
 		(instances
-			(project "watering-system"
+			(project "main-board"
 				(path "/37f9ca20-4a6d-426d-a8d5-c655e0adba86"
 					(reference "#PWR025")
@@
 		)
 		(instances
-			(project "watering-system"
+			(project "main-board"
 				(path "/37f9ca20-4a6d-426d-a8d5-c655e0adba86"
 					(reference "U2")
@@
 		)
 		(instances
-			(project "watering-system"
+			(project "main-board"
 				(path "/37f9ca20-4a6d-426d-a8d5-c655e0adba86"
 					(reference "#PWR01")
@@
 		)
 		(instances
-			(project "watering-system"
+			(project "main-board"
 				(path "/37f9ca20-4a6d-426d-a8d5-c655e0adba86"
 					(reference "#FLG02")
@@
 		)
 		(instances
-			(project "watering-system"
+			(project "main-board"
 				(path "/37f9ca20-4a6d-426d-a8d5-c655e0adba86"
 					(reference "J4")
@@
 		)
 		(instances
-			(project "watering-system"
+			(project "main-board"
 				(path "/37f9ca20-4a6d-426d-a8d5-c655e0adba86"
 					(reference "#PWR031")
@@
 		)
 		(instances
-			(project "watering-system"
+			(project "main-board"
 				(path "/37f9ca20-4a6d-426d-a8d5-c655e0adba86"
 					(reference "#PWR018")
@@
 		)
 		(instances
-			(project "watering-system"
+			(project "main-board"
 				(path "/37f9ca20-4a6d-426d-a8d5-c655e0adba86"
 					(reference "#PWR024")
@@
 		)
 		(instances
-			(project "watering-system"
+			(project "main-board"
 				(path "/37f9ca20-4a6d-426d-a8d5-c655e0adba86"
 					(reference "#PWR08")
@@
 		)
 		(instances
-			(project "watering-system"
+			(project "main-board"
 				(path "/37f9ca20-4a6d-426d-a8d5-c655e0adba86"
 					(reference "#PWR021")
@@
 		)
 		(instances
-			(project "watering-system"
+			(project "main-board"
 				(path "/37f9ca20-4a6d-426d-a8d5-c655e0adba86"
 					(reference "#PWR023")
@@
 		)
 		(instances
-			(project "watering-system"
+			(project "main-board"
 				(path "/37f9ca20-4a6d-426d-a8d5-c655e0adba86"
 					(reference "J3")
@@
 		)
 		(instances
-			(project "watering-system"
+			(project "main-board"
 				(path "/37f9ca20-4a6d-426d-a8d5-c655e0adba86"
 					(reference "#FLG01")
@@
 		)
 		(instances
-			(project "watering-system"
+			(project "main-board"
 				(path "/37f9ca20-4a6d-426d-a8d5-c655e0adba86"
 					(reference "#PWR020")
@@
 		)
 		(instances
-			(project "watering-system"
+			(project "main-board"
 				(path "/37f9ca20-4a6d-426d-a8d5-c655e0adba86"
 					(reference "D2")
@@
 		)
 		(instances
-			(project "watering-system"
+			(project "main-board"
 				(path "/37f9ca20-4a6d-426d-a8d5-c655e0adba86"
 					(reference "R8")
@@
 		)
 		(instances
-			(project "watering-system"
+			(project "main-board"
 				(path "/37f9ca20-4a6d-426d-a8d5-c655e0adba86"
 					(reference "R6")
@@
 		)
 		(instances
-			(project "watering-system"
+			(project "main-board"
 				(path "/37f9ca20-4a6d-426d-a8d5-c655e0adba86"
 					(reference "#PWR015")
@@
 		)
 		(instances
-			(project "watering-system"
+			(project "main-board"
 				(path "/37f9ca20-4a6d-426d-a8d5-c655e0adba86"
 					(reference "#PWR027")
@@
 		)
 		(instances
-			(project "watering-system"
+			(project "main-board"
 				(path "/37f9ca20-4a6d-426d-a8d5-c655e0adba86"
 					(reference "R5")
@@
 		)
 		(instances
-			(project "watering-system"
+			(project "main-board"
 				(path "/37f9ca20-4a6d-426d-a8d5-c655e0adba86"
 					(reference "D1")
@@
 		)
 		(instances
-			(project "watering-system"
+			(project "main-board"
 				(path "/37f9ca20-4a6d-426d-a8d5-c655e0adba86"
 					(reference "D4")
@@
 		)
 		(instances
-			(project "watering-system"
+			(project "main-board"
 				(path "/37f9ca20-4a6d-426d-a8d5-c655e0adba86"
 					(reference "#PWR012")
@@
 		)
 		(instances
-			(project "watering-system"
+			(project "main-board"
 				(path "/37f9ca20-4a6d-426d-a8d5-c655e0adba86"
 					(reference "R7")
@@
 		)
 		(instances
-			(project "watering-system"
+			(project "main-board"
 				(path "/37f9ca20-4a6d-426d-a8d5-c655e0adba86"
 					(reference "#PWR028")
@@
 		)
 		(instances
-			(project "watering-system"
+			(project "main-board"
 				(path "/37f9ca20-4a6d-426d-a8d5-c655e0adba86"
 					(reference "#PWR07")
@@
 		)
 		(instances
-			(project "watering-system"
+			(project "main-board"
 				(path "/37f9ca20-4a6d-426d-a8d5-c655e0adba86"
 					(reference "#PWR026")
@@
 		)
 		(instances
-			(project "watering-system"
+			(project "main-board"
 				(path "/37f9ca20-4a6d-426d-a8d5-c655e0adba86"
 					(reference "#PWR03")
@@
 		)
 		(instances
-			(project "watering-system"
+			(project "main-board"
 				(path "/37f9ca20-4a6d-426d-a8d5-c655e0adba86"
 					(reference "K3")

Commit message: fix: set both light sensor resistors to 10k
Parts:
- R1: value R -> 10k
Changed lines of the file:
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@@
 			)
 		)
-		(property "Value" "R"
+		(property "Value" "10k"
 			(at 229.87 33.0199 0)
 			(show_name no)
